Commit message: separate file for booster ik_reachability

File: src/curobo/content/assets/robot/booster/t1_7dof.urdf (robot description, URDF)
Before this commit: robot T1, 30 links, 29 joints
Links:
- added link left_Link1, mass 0.00647716099397792; collision mesh filename=7_dofs_arms_with_jaw/left_Link1.STL; visual mesh filename=7_dofs_arms_with_jaw/left_Link1.STL
- added link left_Link11, mass 0.0127543420299361; collision mesh filename=7_dofs_arms_with_jaw/left_Link11.STL; visual mesh filename=7_dofs_arms_with_jaw/left_Link11.STL
- added link left_Link2, mass 0.00647716099397793; collision mesh filename=7_dofs_arms_with_jaw/left_Link2.STL; visual mesh filename=7_dofs_arms_with_jaw/left_Link2.STL
- added link left_Link22, mass 0.0127543420299362; collision mesh filename=7_dofs_arms_with_jaw/left_Link22.STL; visual mesh filename=7_dofs_arms_with_jaw/left_Link22.STL
- added link left_base_link, mass 0.105853592307918; collision mesh filename=7_dofs_arms_with_jaw/left_base_link.STL; visual mesh filename=7_dofs_arms_with_jaw/left_base_link.STL
- added link right_Link1, mass 0.00647716099397792; collision mesh filename=7_dofs_arms_with_jaw/right_Link1.STL; visual mesh filename=7_dofs_arms_with_jaw/right_Link1.STL
- added link right_Link11, mass 0.0127543420299361; collision mesh filename=7_dofs_arms_with_jaw/right_Link11.STL; visual mesh filename=7_dofs_arms_with_jaw/right_Link11.STL
- added link right_Link2, mass 0.00647716099397793; collision mesh filename=7_dofs_arms_with_jaw/right_Link2.STL; visual mesh filename=7_dofs_arms_with_jaw/right_Link2.STL
- added link right_Link22, mass 0.0127543420299362; collision mesh filename=7_dofs_arms_with_jaw/right_Link22.STL; visual mesh filename=7_dofs_arms_with_jaw/right_Link22.STL
- added link right_base_link, mass 0.105853592307918; collision mesh filename=7_dofs_arms_with_jaw/right_base_link.STL; visual mesh filename=7_dofs_arms_with_jaw/right_base_link.STL
- link AL1: geometry collision mesh filename=7_dofs_arms_with_jaw/AL1.STL; visual mesh filename=7_dofs_arms_with_jaw/AL1.STL
- link AL2: geometry collision mesh filename=7_dofs_arms_with_jaw/AL2.STL; visual mesh filename=7_dofs_arms_with_jaw/AL2.STL
- link AL3: geometry collision mesh filename=7_dofs_arms_with_jaw/AL3.STL; visual mesh filename=7_dofs_arms_with_jaw/AL3.STL
- link AL4: geometry collision mesh filename=7_dofs_arms_with_jaw/AL4.STL; visual mesh filename=7_dofs_arms_with_jaw/AL4.STL
- link AL5: geometry collision mesh filename=7_dofs_arms_with_jaw/AL5.STL; visual mesh filename=7_dofs_arms_with_jaw/AL5.STL
- link AL6: geometry collision mesh filename=7_dofs_arms_with_jaw/AL6.STL; visual mesh filename=7_dofs_arms_with_jaw/AL6.STL
- link AR1: geometry collision mesh filename=7_dofs_arms_with_jaw/AR1.STL; visual mesh filename=7_dofs_arms_with_jaw/AR1.STL
- link AR2: geometry collision mesh filename=7_dofs_arms_with_jaw/AR2.STL; visual mesh filename=7_dofs_arms_with_jaw/AR2.STL
- link AR3: geometry collision mesh filename=7_dofs_arms_with_jaw/AR3.STL; visual mesh filename=7_dofs_arms_with_jaw/AR3.STL
- link AR4: geometry collision mesh filename=7_dofs_arms_with_jaw/AR4.STL; visual mesh filename=7_dofs_arms_with_jaw/AR4.STL
- link AR5: geometry collision mesh filename=7_dofs_arms_with_jaw/AR5.STL; visual mesh filename=7_dofs_arms_with_jaw/AR5.STL
- link AR6: geometry collision mesh filename=7_dofs_arms_with_jaw/AR6.STL; visual mesh filename=7_dofs_arms_with_jaw/AR6.STL
- link Ankle_Cross_Left: geometry collision mesh filename=7_dofs_arms_with_jaw/Ankle_Cross_Left.STL; visual mesh filename=7_dofs_arms_with_jaw/Ankle_Cross_Left.STL
- link Ankle_Cross_Right: geometry collision mesh filename=7_dofs_arms_with_jaw/Ankle_Cross_Right.STL; visual mesh filename=7_dofs_arms_with_jaw/Ankle_Cross_Right.STL
- link H1: geometry collision mesh filename=7_dofs_arms_with_jaw/H1.STL; visual mesh filename=7_dofs_arms_with_jaw/H1.STL
- link H2: geometry collision mesh filename=7_dofs_arms_with_jaw/H2.STL; visual mesh filename=7_dofs_arms_with_jaw/H2.STL
- link Hip_Pitch_Left: geometry collision mesh filename=7_dofs_arms_with_jaw/Hip_Pitch_Left.STL; visual mesh filename=7_dofs_arms_with_jaw/Hip_Pitch_Left.STL
- link Hip_Pitch_Right: geometry collision mesh filename=7_dofs_arms_with_jaw/Hip_Pitch_Right.STL; visual mesh filename=7_dofs_arms_with_jaw/Hip_Pitch_Right.STL
- link Hip_Roll_Left: geometry collision mesh filename=7_dofs_arms_with_jaw/Hip_Roll_Left.STL; visual mesh filename=7_dofs_arms_with_jaw/Hip_Roll_Left.STL
- link Hip_Roll_Right: geometry collision mesh filename=7_dofs_arms_with_jaw/Hip_Roll_Right.STL; visual mesh filename=7_dofs_arms_with_jaw/Hip_Roll_Right.STL
- link Hip_Yaw_Left: geometry collision mesh filename=7_dofs_arms_with_jaw/Hip_Yaw_Left.STL; visual mesh filename=7_dofs_arms_with_jaw/Hip_Yaw_Left.STL
- link Hip_Yaw_Right: geometry collision mesh filename=7_dofs_arms_with_jaw/Hip_Yaw_Right.STL; visual mesh filename=7_dofs_arms_with_jaw/Hip_Yaw_Right.STL
- link Shank_Left: geometry collision mesh filename=7_dofs_arms_with_jaw/Shank_Left.STL; visual mesh filename=7_dofs_arms_with_jaw/Shank_Left.STL
- link Shank_Right: geometry collision mesh filename=7_dofs_arms_with_jaw/Shank_Right.STL; visual mesh filename=7_dofs_arms_with_jaw/Shank_Right.STL
- link Trunk: geometry collision mesh filename=7_dofs_arms_with_jaw/Trunk.STL; visual mesh filename=7_dofs_arms_with_jaw/Trunk.STL
- link Waist: geometry collision mesh filename=7_dofs_arms_with_jaw/Waist.STL; visual mesh filename=7_dofs_arms_with_jaw/Waist.STL
- link left_foot_link: geometry collision mesh filename=7_dofs_arms_with_jaw/left_foot_link.STL; visual mesh filename=7_dofs_arms_with_jaw/left_foot_link.STL
- link left_hand_link: geometry collision mesh filename=7_dofs_arms_with_jaw/AL7.STL; visual mesh filename=7_dofs_arms_with_jaw/AL7.STL
- link right_foot_link: geometry collision mesh filename=7_dofs_arms_with_jaw/right_foot_link.STL; visual mesh filename=7_dofs_arms_with_jaw/right_foot_link.STL
- link right_hand_link: geometry collision mesh filename=7_dofs_arms_with_jaw/AR7.STL; visual mesh filename=7_dofs_arms_with_jaw/AR7.STL
Joints:
- added joint left_Link1: type revolute, parent left_base_link, child left_Link1, origin xyz=0.036 -0.04 -0.019 rpy=-3.0158E-16 -7.1586E-16 -0.30719, axis 0 1 0, limit lower=0 upper=1 effort=1 velocity=1
- added joint left_Link11: type revolute, parent left_Link1, child left_Link11, origin xyz=0.042 0 0.003 rpy=5.0393E-16 5.6225E-16 0.30719, axis 0 1 0, limit lower=-1 upper=0 effort=1 velocity=1
- added joint left_Link2: type revolute, parent left_base_link, child left_Link2, origin xyz=0.036 0.04 -0.019 rpy=-2.6397E-16 3.7199E-16 0.30719, axis 0 1 0, limit lower=-1 upper=0 effort=1 velocity=1
- added joint left_Link22: type revolute, parent left_Link2, child left_Link22, origin xyz=0.042 0 0.015 rpy=-3.641E-16 2.4584E-16 2.8344, axis 0 1 0, limit lower=0 upper=1 effort=1 velocity=1
- added joint left_base_link: type fixed, parent left_hand_link, child left_base_link, origin xyz=-0.006 0.08 0.01 rpy=0 0 1.5708, axis 1 0 0, limit lower=0 upper=1 effort=1 velocity=1
- added joint right_Link1: type revolute, parent right_base_link, child right_Link1, origin xyz=0.036 -0.04 -0.019 rpy=0 0 -0.30719, axis 0 1 0, limit lower=0 upper=1 effort=1 velocity=1
- added joint right_Link11: type revolute, parent right_Link1, child right_Link11, origin xyz=0.042 0 0.003 rpy=5.0393E-16 5.6225E-16 0.30719, axis 0 1 0, limit lower=-1 upper=0 effort=1 velocity=1
- added joint right_Link2: type revolute, parent right_base_link, child right_Link2, origin xyz=0.036 0.04 -0.019 rpy=-2.6397E-16 3.7199E-16 0.30719, axis 0 1 0, limit lower=-1 upper=0 effort=1 velocity=1
- added joint right_Link22: type revolute, parent right_Link2, child right_Link22, origin xyz=0.042 0 0.015 rpy=-3.641E-16 2.4584E-16 2.8344, axis 0 1 0, limit lower=0 upper=1 effort=1 velocity=1
- added joint right_base_link: type fixed, parent right_hand_link, child right_base_link, origin xyz=-0.006 -0.084 0.01 rpy=0 0 -1.5708, axis 1 0 0, limit lower=0 upper=1 effort=1 velocity=1
- joint AAHead_yaw: limit lower=-1.57 upper=1.57 effort=7 velocity=12.56 -> lower=-1.012 upper=1.012 effort=100 velocity=50
- joint Head_pitch: limit lower=-0.35 upper=1.22 effort=7 velocity=12.56 -> lower=-0.314 upper=0.82 effort=100 velocity=50
- joint Left_Ankle_Pitch: limit lower=-0.87 upper=0.35 effort=12 velocity=18.8 -> lower=-1.57 upper=1.57 effort=100 velocity=50
- joint Left_Ankle_Roll: limit lower=-0.44 upper=0.44 effort=12 velocity=12.4 -> lower=-1.57 upper=1.57 effort=100 velocity=50
- joint Left_Elbow_Pitch: limit lower=-2.27 upper=2.27 effort=18 velocity=18.84 -> lower=-3.14 upper=3.14 effort=100 velocity=50
- joint Left_Elbow_Yaw: limit lower=-2.27 upper=2.27 effort=18 velocity=18.84 -> lower=-3.14 upper=3.14 effort=100 velocity=50
- joint Left_Hand_Roll: limit lower=-2.27 upper=2.27 effort=18 velocity=18.84 -> lower=-3.14 upper=3.14 effort=100 velocity=50
- joint Left_Hip_Pitch: limit lower=-1.8 upper=1.57 effort=45 velocity=12.5 -> lower=-1.57 upper=1.57 effort=100 velocity=50
- joint Left_Hip_Roll: limit lower=-0.3 upper=1.57 effort=30 velocity=10.9 -> lower=-1.57 upper=1.57 effort=100 velocity=50
- joint Left_Hip_Yaw: limit lower=-1 upper=1 effort=30 velocity=10.9 -> lower=-1.57 upper=1.57 effort=100 velocity=50
- joint Left_Knee_Pitch: limit lower=0 upper=2.34 effort=60 velocity=11.7 -> lower=-1.57 upper=1.57 effort=100 velocity=50
- joint Left_Shoulder_Pitch: limit lower=-3.31 upper=1.22 effort=18 velocity=18.84 -> lower=-3.28 upper=1.186 effort=100 velocity=50
- joint Left_Shoulder_Roll: limit lower=-1.74 upper=1.57 effort=18 velocity=18.84 -> lower=-1.64 upper=1.535 effort=100 velocity=50
- joint Left_Wrist_Pitch: limit lower=-2.27 upper=2.27 effort=18 velocity=18.84 -> lower=-3.14 upper=3.14 effort=100 velocity=50
- joint Left_Wrist_Yaw: limit lower=-2.27 upper=2.27 effort=18 velocity=18.84 -> lower=-3.14 upper=3.14 effort=100 velocity=50
- joint Right_Ankle_Pitch: limit lower=-0.87 upper=0.35 effort=12 velocity=18.8 -> lower=-1.57 upper=1.57 effort=100 velocity=50
- joint Right_Ankle_Roll: limit lower=-0.44 upper=0.44 effort=12 velocity=12.4 -> lower=-1.57 upper=1.57 effort=100 velocity=50
- joint Right_Elbow_Pitch: limit lower=-2.27 upper=2.27 effort=18 velocity=18.84 -> lower=-1.57 upper=1.57 effort=100 velocity=50
- joint Right_Elbow_Yaw: limit lower=-2.27 upper=2.27 effort=18 velocity=18.84 -> lower=-1.57 upper=1.57 effort=100 velocity=50
- joint Right_Hand_Roll: limit lower=-2.27 upper=2.27 effort=18 velocity=18.84 -> lower=-1.57 upper=1.57 effort=100 velocity=50
- joint Right_Hip_Pitch: limit lower=-1.8 upper=1.57 effort=45 velocity=12.5 -> lower=-1.57 upper=1.57 effort=100 velocity=50
- joint Right_Hip_Roll: limit lower=-1.57 upper=0.3 effort=30 velocity=10.9 -> lower=-1.57 upper=1.57 effort=100 velocity=50
- joint Right_Hip_Yaw: limit lower=-1 upper=1 effort=30 velocity=10.9 -> lower=-1.57 upper=1.57 effort=100 velocity=50
- joint Right_Knee_Pitch: limit lower=0 upper=2.34 effort=60 velocity=11.7 -> lower=-1.57 upper=1.57 effort=100 velocity=50
- joint Right_Shoulder_Pitch: limit lower=-3.31 upper=1.22 effort=18 velocity=18.84 -> lower=-1.57 upper=1.57 effort=100 velocity=50
- joint Right_Shoulder_Roll: limit lower=-1.57 upper=1.74 effort=18 velocity=18.84 -> lower=-1.57 upper=1.57 effort=100 velocity=50
- joint Right_Wrist_Pitch: limit lower=-2.27 upper=2.27 effort=18 velocity=18.84 -> lower=-1.57 upper=1.57 effort=100 velocity=50
- joint Right_Wrist_Yaw: limit lower=-2.27 upper=2.27 effort=18 velocity=18.84 -> lower=-1.57 upper=1.57 effort=100 velocity=50
- joint Waist: limit lower=-1.57 upper=1.57 effort=30 velocity=10.88 -> lower=-1.57 upper=1.57 effort=100 velocity=50

Commit message: urdf path fixed

File: src/curobo/content/assets/robot/booster/t1_7dof.urdf (robot description, URDF)
Before this commit: robot V23RobotAsm, 40 links, 39 joints
Links:
- link AL1: geometry collision mesh filename=meshes/AL1.STL; visual mesh filename=meshes/AL1.STL
- link AL2: geometry collision mesh filename=meshes/AL2.STL; visual mesh filename=meshes/AL2.STL
- link AL3: geometry collision mesh filename=meshes/AL3.STL; visual mesh filename=meshes/AL3.STL
- link AL4: geometry collision mesh filename=meshes/AL4.STL; visual mesh filename=meshes/AL4.STL
- link AL5: geometry collision mesh filename=meshes/AL5.STL; visual mesh filename=meshes/AL5.STL
- link AL6: geometry collision mesh filename=meshes/AL6.STL; visual mesh filename=meshes/AL6.STL
- link AR1: geometry collision mesh filename=meshes/AR1.STL; visual mesh filename=meshes/AR1.STL
- link AR2: geometry collision mesh filename=meshes/AR2.STL; visual mesh filename=meshes/AR2.STL
- link AR3: geometry collision mesh filename=meshes/AR3.STL; visual mesh filename=meshes/AR3.STL
- link AR4: geometry collision mesh filename=meshes/AR4.STL; visual mesh filename=meshes/AR4.STL
- link AR5: geometry collision mesh filename=meshes/AR5.STL; visual mesh filename=meshes/AR5.STL
- link AR6: geometry collision mesh filename=meshes/AR6.STL; visual mesh filename=meshes/AR6.STL
- link Ankle_Cross_Left: geometry collision mesh filename=meshes/Ankle_Cross_Left.STL; visual mesh filename=meshes/Ankle_Cross_Left.STL
- link Ankle_Cross_Right: geometry collision mesh filename=meshes/Ankle_Cross_Right.STL; visual mesh filename=meshes/Ankle_Cross_Right.STL
- link H1: geometry collision mesh filename=meshes/H1.STL; visual mesh filename=meshes/H1.STL
- link H2: geometry collision mesh filename=meshes/H2.STL; visual mesh filename=meshes/H2.STL
- link Hip_Pitch_Left: geometry collision mesh filename=meshes/Hip_Pitch_Left.STL; visual mesh filename=meshes/Hip_Pitch_Left.STL
- link Hip_Pitch_Right: geometry collision mesh filename=meshes/Hip_Pitch_Right.STL; visual mesh filename=meshes/Hip_Pitch_Right.STL
- link Hip_Roll_Left: geometry collision mesh filename=meshes/Hip_Roll_Left.STL; visual mesh filename=meshes/Hip_Roll_Left.STL
- link Hip_Roll_Right: geometry collision mesh filename=meshes/Hip_Roll_Right.STL; visual mesh filename=meshes/Hip_Roll_Right.STL
- link Hip_Yaw_Left: geometry collision mesh filename=meshes/Hip_Yaw_Left.STL; visual mesh filename=meshes/Hip_Yaw_Left.STL
- link Hip_Yaw_Right: geometry collision mesh filename=meshes/Hip_Yaw_Right.STL; visual mesh filename=meshes/Hip_Yaw_Right.STL
- link Shank_Left: geometry collision mesh filename=meshes/Shank_Left.STL; visual mesh filename=meshes/Shank_Left.STL
- link Shank_Right: geometry collision mesh filename=meshes/Shank_Right.STL; visual mesh filename=meshes/Shank_Right.STL
- link Trunk: geometry collision mesh filename=meshes/Trunk.STL; visual mesh filename=meshes/Trunk.STL
- link Waist: geometry collision mesh filename=meshes/Waist.STL; visual mesh filename=meshes/Waist.STL
- link left_Link1: geometry collision mesh filename=meshes/left_Link1.STL; visual mesh filename=meshes/left_Link1.STL
- link left_Link11: geometry collision mesh filename=meshes/left_Link11.STL; visual mesh filename=meshes/left_Link11.STL
- link left_Link2: geometry collision mesh filename=meshes/left_Link2.STL; visual mesh filename=meshes/left_Link2.STL
- link left_Link22: geometry collision mesh filename=meshes/left_Link22.STL; visual mesh filename=meshes/left_Link22.STL
- link left_base_link: geometry collision mesh filename=meshes/left_base_link.STL; visual mesh filename=meshes/left_base_link.STL
- link left_foot_link: geometry collision mesh filename=meshes/left_foot_link.STL; visual mesh filename=meshes/left_foot_link.STL
- link left_hand_link: geometry collision mesh filename=meshes/AL7.STL; visual mesh filename=meshes/AL7.STL
- link right_Link1: geometry collision mesh filename=meshes/right_Link1.STL; visual mesh filename=meshes/right_Link1.STL
- link right_Link11: geometry collision mesh filename=meshes/right_Link11.STL; visual mesh filename=meshes/right_Link11.STL
- link right_Link2: geometry collision mesh filename=meshes/right_Link2.STL; visual mesh filename=meshes/right_Link2.STL
- link right_Link22: geometry collision mesh filename=meshes/right_Link22.STL; visual mesh filename=meshes/right_Link22.STL
- link right_base_link: geometry collision mesh filename=meshes/right_base_link.STL; visual mesh filename=meshes/right_base_link.STL
- link right_foot_link: geometry collision mesh filename=meshes/right_foot_link.STL; visual mesh filename=meshes/right_foot_link.STL
- link right_hand_link: geometry collision mesh filename=meshes/AR7.STL; visual mesh filename=meshes/AR7.STL
